Commit message: some cleaning up

File: panos_bot/urdf/panos_bot.xacro (robot description, xacro)
@@ -59,7 +59,4 @@
     </visual>
   </link>
-  <gazebo reference="chassis">
-    <material>Gazebo/Green</material>
-  </gazebo>
   <!-- sensor base -->
   <link name='sensor_base'>
@@ -85,11 +82,9 @@
         <box size=".15 .15 .25"/>
       </geometry>
-    </visual>
-  </link>
-  <joint type="fixed" name="sensor_base_joint">
-    <origin xyz="0 0 0" rpy="0 0 0"/>
-    <child link="sensor_base"/>
-    <parent link="chassis"/>
-  </joint>
+      <material name="black">
+        <color rgba="0 0 0 1"/>
+      </material>
+    </visual>
+  </link>
   <!-- Left Wheel Link -->
   <link name="left_wheel">
@@ -119,7 +114,4 @@
     </collision>
   </link>
-  <gazebo reference="left_wheel">
-    <material>Gazebo/Blue</material>
-  </gazebo>
   <!-- Right Wheel Link -->
   <link name="right_wheel">
@@ -149,7 +141,4 @@
     </collision>
   </link>
-  <gazebo reference="right_wheel">
-    <material>Gazebo/Blue</material>
-  </gazebo>
   <!-- Camera Link -->
   <link name="camera">
@@ -179,7 +168,4 @@
     </collision>
   </link>
-  <gazebo reference="camera">
-    <material>Gazebo/Yellow</material>
-  </gazebo>
   <!-- Hokuyo Link -->
   <link name="hokuyo">
@@ -209,7 +195,4 @@
     </collision>
   </link>
-  <gazebo reference="hokuyo">
-    <material>Gazebo/Red</material>
-  </gazebo>
   <!-- Joints -->
   <joint type="continuous" name="left_wheel_hinge">
@@ -239,3 +222,8 @@
     <parent link="sensor_base"/>
   </joint>
+  <joint type="fixed" name="sensor_base_joint">
+    <origin xyz="0 0 0" rpy="0 0 0"/>
+    <child link="sensor_base"/>
+    <parent link="chassis"/>
+  </joint>
 </robot>
